File: Electronics/axis_control_board/axis_control_board.kicad_pcb (KiCad board)
At the start: 2 copper layers, 58.2 x 63.2 mm, 28 parts, among them Q1 S8050, U1 LD33v_TO220, U2 NRF24L01_Breakout, U4 LM7805_TO220

Commit message: updated axis_control PCB and fixed hardware bug
Parts:
- removed U1: LD33v_TO220, Package_TO_SOT_THT:TO-220-3_Vertical
- added Bridge5: 0ohm, Resistor_THT:R_Axial_DIN0207_L6.3mm_D2.5mm_P5.08mm_Vertical, F.Cu at (173.8, 130.6)
- added U3: AMS1117-3.3, Package_TO_SOT_THT:TO-220-3_Vertical, F.Cu at (169.9, 133.9)
- A1, A2: value Pololu_Breakout_DRV8825 -> DRV8825
- Debug_Pinout1, TOF_sensor1: value Conn_01x03_Socket -> 01x03
- Power_in1: value Conn_01x02_Socket -> JST-2P
- R2: value 1k -> 2k
- STC8H8K64U1: value Conn_02x14_Counter_Clockwise -> SKDIP28
Connections:
- STC8H8K64U1 pad 2: unconnected-(STC8H8K64U1-Pin_2-Pad2) -> CSN
- STC8H8K64U1 pad 8: CSN -> unconnected-(STC8H8K64U1-Pin_8-Pad8)
Routing:
- net CSN: track 14.9 -> 26.3 mm
- net GND: track 196.2 -> 205.9 mm
- net +3.3V: track 228.7 -> 234.0 mm
- net Net-(U3-VO): track 0.00 -> 4.24 mm

Commit message: finished sensor board PCB
Parts:
- Stepper_motor1, Stepper_motor2: value Conn_01x04_Socket -> JST4P
- TOF1: renamed from TOF_sensor1; value 01x03 -> 1x3
- Ultrasonic_Pinout1: value Conn_01x04_Socket -> JST_4P
Routing:
- net +3.3V: track 234.0 -> 239.7 mm
- net Net-(Q1-B): track 9.30 -> 12.7 mm
- net +5V: track 59.4 -> 62.1 mm
- net +12V: track 83.7 -> 84.4 mm
- net GND: track 205.9 -> 206.5 mm
