File: Electronics/Main_board/Main_board.kicad_pcb (KiCad board)
At the start: 2 copper layers, 39 parts, among them Q1 S8050, Q2 S8050, Q3 IRFZ44n, Q4 IRFZ44n, Q5 IRFZ44n, U1 AMS1117-3.3, U2 NRF24L01_Breakout, U3 LM7805_TO220, U4 PC817, U5 PC817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

Commit message: finished Main Board PCB
Parts:
- added H1: MountingHole, MountingHole:MountingHole_3.2mm_M3_DIN965_Pad_TopBottom, F.Cu at (91.0, 72.0)
- added H2: MountingHole, MountingHole:MountingHole_3.2mm_M3_DIN965_Pad_TopBottom, F.Cu at (167.0, 72.0)
- moved U2 77.4 mm to (162.7, 138.9), turned to 180 degrees
- moved C2 66.2 mm to (93.2, 128.7), turned to -90 degrees
- moved R1 64.8 mm to (168.3, 86.0), turned to 180 degrees
- moved R6 63.1 mm to (168.3, 83.0), turned to 180 degrees
- moved WaterChannel1 60.0 mm to (96.5, 81.0), turned to 180 degrees
- moved WaterChannel2 55.9 mm to (105.1, 80.4)
- moved C1 51.6 mm to (101.4, 137.9), turned to 90 degrees
- moved Power12V1 50.4 mm to (93.2, 137.6), turned to 90 degrees
- moved R2 49.2 mm to (149.3, 96.2)
- moved UART1 48.6 mm to (90.4, 122.9)
- moved R3 46.9 mm to (151.8, 85.5), turned to -90 degrees
- moved R4 42.5 mm to (146.6, 93.2), turned to 90 degrees
- moved CAN_line1 40.1 mm to (165.4, 100.8), turned to -90 degrees
- moved Q4 40.0 mm to (105.6, 116.6), turned to 90 degrees
- moved C3 38.0 mm to (121.8, 134.0), turned to 90 degrees
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Connections:
- Pico_W1 pad 19: CRX_3.3v -> unconnected-(Pico_W1-Pin_19-Pad19)
- Pico_W1 pad 20: CTX_3.3v -> unconnected-(Pico_W1-Pin_20-Pad20)
- Pico_W2 pad 10: unconnected-(Pico_W2-Pin_10-Pad10) -> CTX_3.3v
- Pico_W2 pad 13: unconnected-(Pico_W2-Pin_13-Pad13) -> GND
- Pico_W2 pad 9: unconnected-(Pico_W2-Pin_9-Pad9) -> CRX_3.3v
Routing:
- net GND: track 0.00 -> 468.4 mm
- net +5V: track 0.00 -> 182.2 mm
- net +3.3V: track 0.00 -> 171.4 mm
- net +12V: track 0.00 -> 104.9 mm
- net CTX: track 0.00 -> 68.8 mm
- net TX: track 0.00 -> 55.8 mm
- net CSN: track 0.00 -> 44.8 mm
- net CRX: track 0.00 -> 44.1 mm
- net CE: track 0.00 -> 41.2 mm
- net MOSI: track 0.00 -> 38.5 mm
- net R1A: track 0.00 -> 36.2 mm
- net R2A: track 0.00 -> 33.7 mm
- net SCK: track 0.00 -> 32.9 mm
- net R3A: track 0.00 -> 31.5 mm
- net R3B: track 0.00 -> 24.9 mm
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Other:
- board text added: "SIMACAS Main Board"

Commit message: added Main Board PDFs
Other:
- board outline added: 87.2 x 81.7 mm
Changed lines of the file:
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@@
     )
   )
+  (gr_rect (start 85.33 60.96) (end 172.56 142.68)
+    (stroke (width 0.2) (type default)) (fill none) (layer "Edge.Cuts"))
   (gr_rect (start 148.79 109.05) (end 167.79 125.05)
     (stroke (width 0.2) (type default)) (fill none) (layer "F.Fab"))
-  (gr_rect (start 85.33 60.96) (end 172.56 142.68)
-    (stroke (width 0.2) (type default)) (fill none) (layer "F.Fab"))
   (gr_text "SIMACAS Main Board" (at 89.53 67.93) (layer "F.Fab")
